File: led_driver_12v_1a_32mm.sch (EAGLE design)
At the start: 44 parts, among them IC1 LM2936MP-3.0, Q1 BSZ0902NSI, Q2 BSZ0902NSI, Q3 BSZ0902NSI, Q4 BSZ0902NSI, Q5 BSZ0902NSI, X1 87758-1016

Commit message: Restores 32mm version
Parts:
- removed IC1: LM2936MP-3.0, national-semiconductor:LM2936MP-3.0
- removed X1: 87758-1016, con-molex:87758-1016
- added D1: BAT46-WJ, diode:DIODE-SOD323-W
- added INT0: TPTP20SQ, testpad:TPTP20SQ
- added MISO, MOSI, RST, SCK, VCC: TPTP11R, testpad:TPTP11R
- added PAD5: GND, wirepad:WIREPADSMD1,27-254
- added Q6: SSM3K2615R, SparkFun-DiscreteSemi:MOSFET-NCHANNELBSS123LT1G
- added R1: 10k, resistor:R-EU_R0402
- added R2: 300k, resistor:R-EU_R0402
- added R3: 56.9k, resistor:R-EU_R0402
- C16: value 10uF -> 4.7uF
- PAD1, PAD2: device wirepad:WIREPAD3,81/1,4 -> wirepad:WIREPADSMD5-2,5
Connections:
- removed net N$10: U$1.EN/ULVO, U$2.PB0
- removed net N$22: U$2.PB3/RESET, X1-4.S
- removed net N$23: U$2.PB2, X1-3.S
- removed net N$8: U$2.PA1/ADC1, X1-10.S
- net +12V: now also Q6.G, R2.2; no longer IC1.VIN
- net DGND: now also Q6.S, R10.1, R3.1; no longer IC1.GND@1, IC1.GND@2
- net GND: now also PAD5.P; no longer R10.1
- net INTVCC: now also D1.A
- net N$11: now also R2.1, R3.2, U$1.EN/ULVO; no longer U$2.PA2/ADC2, X1-9.S
- net N$12: now also D1.C, R1.1, VCC.TP; no longer IC1.VO, X1-2.S
- net N$13: now also INT0.TP, Q6.D, R1.2, U$2.PB2; no longer U$2.PA3/ADC3, X1-8.S
- net N$16: now also MISO.TP, U$2.PA5/MISO; no longer U$2.PA4/SCL, X1-7.S
- net N$17: now also MOSI.TP, U$2.PA6/MOSI; no longer U$2.PA5/MISO, X1-6.S
- net N$18: now also RST.TP, U$2.PB3/RESET; no longer U$2.PA6/MOSI, X1-5.S
- net N$20: now also SCK.TP, U$2.PA4/SCL; no longer U$2.PB1, X1-1.S
Other:
- note removed: "The ESR, of the COUT capacitor must at least 300 mΩ, but no more than 8 Ω"
- note removed: "WARNING! SOLDER R8 TO GROUND MANUALLY!"
- moved on the sheet: R5, R6
