File: rect_and_stab/charger.sch (EAGLE design)
At the start: 92 parts, among them Q1 BSZ0902NSI, Q2 BSZ0902NSI, Q3 FDN360P, Q4 BSZ0902NSI, Q5 BSZ0902NSI, Q6 BSS138, Q7 MOSFET-NCHANNEL2N7002PW, Q8 BSZ0902NSI, Q9 BSS138

Commit message: board routed and secondary protection removed
Parts:
- removed C23, C24, C25, C26, C27, C28: 0.1uF, resistor:C-EUC0402
- removed Q6: BSS138, SparkFun-DiscreteSemi:MOSFET-NCHANNEL2N7002PW
- removed R30: 5.1k, resistor:R-EU_R0402
- removed R32, R33, R34: 1k, resistor:R-EU_R0402
- removed R35: 100, resistor:R-EU_R0402
- removed R36: 20k, resistor:R-EU_R0402
- removed U$17: SCP, SCP:SCP
- removed U$9: BQ2947, bq2947:BQ2947
- C9: value 1.5uF -> 2.2uF
- R25: device resistor:R-EU_R2512 -> resistor:R-EU_R2010
Connections:
- removed net N$46: C23.1, U$9.CD
- removed net N$47: R30.1, R31.1, R36.2
- removed net N$48: R30.2, U$9.OUT
- removed net N$49: C25.2, C26.1, R33.1, U$9.V2
- removed net N$50: C26.2, C27.1, R34.1, U$9.V1
- removed net N$51: C25.1, R32.1, U$9.V3, U$9.V4
- removed net N$52: Q6.D, U$17.4
- removed net N$53: C24.1, R35.2, U$9.VDD
- removed net N$55: C28.2, Q6.G, R36.1
- net AGND: no longer C23.2, C24.2, C27.2, C28.1, Q6.S, U$9.PWPD, U$9.VSS
- net GND: now also R31.1
- net N$26: no longer U$17.3
- net N$3: no longer R34.2
- net N$7: no longer R32.2, R35.1, U$17.1
- net N$8: no longer R33.2
